File: OPA564 Voltage Follower.kicad_pcb (KiCad board)
At the start: 2 copper layers, 20 parts, among them IC1 OPA564AIDWD, IC2 OPA564AIDWD, J1 Conn_Coaxial, J2 Conn_Coaxial

Commit message: fixed everything
Parts:
- renumbered REF** to R0
Routing:
- net -12 Volts: track 114.2 -> 112.9 mm
Other:
- board outline added: 70 x 45 mm
- board text added: "Function Amplifier w/ Voltage Follower Andy Yang"
Changed lines of the file:
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@@
 		(descr "Resistor SMD 0603 (1608 Metric), square (rectangular) end terminal, IPC-7351 nominal with elongated pad for handsoldering. (Body size source: IPC-SM-782 page 72, https://www.pcb-3d.com/wordpress/wp-content/uploads/ipc-sm-782a_amendment_1_and_2.pdf)")
 		(tags "resistor handsolder")
-		(property "Reference" "REF**"
-			(at 0 -1.43 0)
+		(property "Reference" "R0"
+			(at -0.5 -1.5 0)
 			(layer "F.SilkS")
 			(effects
@@
 		)
 		(property "Value" "0 Ohm"
-			(at 0 1.43 0)
+			(at -4.5 -1.5 0)
 			(layer "F.Fab")
 			(effects
@@
 		(tags "resistor handsolder")
 		(property "Reference" "R1"
-			(at 0 -1.65 90)
+			(at -3 0 180)
 			(layer "F.SilkS")
 			(effects
@@
 		(descr "Resistor SMD 0603 (1608 Metric), square (rectangular) end terminal, IPC-7351 nominal with elongated pad for handsoldering. (Body size source: IPC-SM-782 page 72, https://www.pcb-3d.com/wordpress/wp-content/uploads/ipc-sm-782a_amendment_1_and_2.pdf)")
 		(tags "resistor handsolder")
-		(property "Reference" "REF**"
-			(at 0 -1.43 90)
+		(property "Reference" "R0"
+			(at -3.0875 0 90)
 			(layer "F.SilkS")
 			(effects
@@
 		(tags "resistor handsolder")
 		(property "Reference" "R2"
-			(at 0 -1.65 90)
+			(at 2.5 0 180)
 			(layer "F.SilkS")
 			(effects
@@
 		(tags "resistor handsolder")
 		(property "Reference" "R3"
-			(at 0 -1.65 90)
+			(at 2.5 0 180)
 			(layer "F.SilkS")
 			(effects
@@
 		(descr "Resistor SMD 0603 (1608 Metric), square (rectangular) end terminal, IPC-7351 nominal with elongated pad for handsoldering. (Body size source: IPC-SM-782 page 72, https://www.pcb-3d.com/wordpress/wp-content/uploads/ipc-sm-782a_amendment_1_and_2.pdf)")
 		(tags "resistor handsolder")
-		(property "Reference" "REF**"
-			(at 0 -1.43 90)
+		(property "Reference" "R0"
+			(at 2.5 0 180)
 			(layer "F.SilkS")
 			(effects
@@
 		)
 	)
+	(gr_rect
+		(start 132.5 45)
+		(end 202.5 90)
+		(stroke
+			(width 0.05)
+			(type default)
+		)
+		(fill no)
+		(layer "Edge.Cuts")
+	)
+	(gr_text "Function Amplifier w/ Voltage Follower\nAndy Yang\n"
+		(at 134 88.5 0)
+		(layer "Edge.Cuts")
+		(effects
+			(font
+				(size 1 1)
+				(thickness 0.15)
+			)
+			(justify left bottom)
+		)
+	)
 	(segment
 		(start 159.269 61.5)
@@
 	)
 	(segment
-		(start 161.5 62.5)
-		(end 162 62.5)
-		(width 0.2)
-		(layer "F.Cu")
-		(net "-12 Volts")
-	)
-	(segment
 		(start 159.199 61.43)
 		(end 160.43 61.43)
@@
 	)
 	(segment
-		(start 177.5 61.77)
-		(end 177.77 61.77)
+		(start 161.5 62.5)
+		(end 161.9625 62.0375)
 		(width 0.2)
 		(layer "F.Cu")
@@
 	)
 	(segment
-		(start 162.73 61.77)
-		(end 168.102 61.77)
+		(start 177.5 61.77)
+		(end 177.77 61.77)
 		(width 0.2)
 		(layer "F.Cu")
@@
 	)
 	(segment
+		(start 161.9625 62.0375)
+		(end 166.5025 62.0375)
+		(width 0.2)
+		(layer "F.Cu")
+		(net "-12 Volts")
+	)
+	(segment
 		(start 152 50.5)
 		(end 152 57)
@@
 	)
 	(segment
-		(start 162 62.5)
-		(end 162.73 61.77)
-		(width 0.2)
-		(layer "F.Cu")
-		(net "-12 Volts")
-	)
-	(segment
 		(start 166.5 59.5)
 		(end 166.77 59.23)
@@
 	)
 	(segment
+		(start 166.5025 62.0375)
+		(end 166.77 61.77)
+		(width 0.2)
+		(layer "F.Cu")
+		(net "-12 Volts")
+	)
+	(segment
 		(start 170 51)
 		(end 170 57.332)
@@
 	)
 	(segment
-		(start 180.5 49.9)
-		(end 180.5 50.5)
+		(start 179.8 50.5)
+		(end 179.5 50.2)
 		(width 0.2)
 		(layer "F.Cu")
@@
 	)
 	(segment
-		(start 179.1 48.5)
-		(end 180.5 49.9)
+		(start 180.5 50.5)
+		(end 179.8 50.5)
+		(width 0.2)
+		(layer "F.Cu")
+		(net "Signal Output")
+	)
+	(segment
+		(start 179.5 49)
+		(end 179 48.5)
 		(width 0.2)
 		(layer "F.Cu")
@@
 	(segment
 		(start 166.934315 48.5)
-		(end 179.1 48.5)
+		(end 179 48.5)
 		(width 0.2)
 		(layer "F.Cu")
@@
 		(width 0.2)
 		(layer "F.Cu")
+		(net "Signal Output")
+	)
+	(segment
+		(start 179.5 50.2)
+		(end 179.5 49)
+		(width 0.2)
+		(layer "F.Cu")

Commit message: version 1 i guess
Routing:
- added copper zone on F.Cu, net GND
Other:
- board text removed: "Function Amplifier w/ Voltage Follower Andy Yang"
Changed lines of the file:
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@@
 		(layer "Edge.Cuts")
-	)
-	(gr_text "Function Amplifier w/ Voltage Follower\nAndy Yang\n"
-		(at 134 88.5 0)
-		(layer "Edge.Cuts")
-		(effects
-			(font
-				(size 1 1)
-				(thickness 0.15)
-			)
-			(justify left bottom)
-		)
 	)
 	(segment
@@
 		(net "Net-(IC2-ISET)")
 	)
+	(zone
+		(net "GND")
+		(layer "F.Cu")
+		(hatch edge 0.5)
+		(connect_pads
+			(clearance 0.5)
+		)
+		(min_thickness 0.25)
+		(fill yes
+			(thermal_gap 0.5)
+			(thermal_bridge_width 0.5)
+			(island_removal_mode 0)
+		)
+		(polygon
+			(pts
+				(xy 202.5 90) (xy 202.5 45) (xy 132.5 45) (xy 132.5 90)
+			)
+		)
+	)
 	(embedded_fonts no)
